Commit message: add finger TF

File: catkin_ws/src/bsl_plotter_description/urdf/bsl_plotter.xacro (robot description, xacro)
@@ -84,4 +84,11 @@
   </collision>
 </link>
+<link name="link_finger">
+  <inertial>
+    <origin xyz="0.0 0.0 0.0" rpy="0 0 0"/>
+    <mass value="0.18190095498276979"/>
+    <inertia ixx="0.000195" iyy="0.000198" izz="3.4e-05" ixy="-0.0" iyz="-1e-06" ixz="-2.6e-05"/>
+  </inertial>
+</link>
 <joint name="rev1" type="continuous">
   <origin xyz="0.0 0.0 0.012628" rpy="0 0 0"/>
@@ -102,3 +109,9 @@
   <axis xyz="0.0 -1.0 -0.0"/>
 </joint>
+<joint name="rev4" type="continuous">
+  <origin xyz="0.225 0.0186 0.0" rpy="0 0 0"/>
+  <parent link="link_hand_v9_1"/>
+  <child link="link_finger"/>
+  <axis xyz="0.0 -1.0 -0.0"/>
+</joint>
 </robot>
